File: PCB/smartBall/GSM_sheet.kicad_sch (KiCad schematic)
At the start: 19 parts, among them IC13 TXB0108PWR, J6 SIM8055-6-1-14-00-A, J7 FXP612 (u.FL) 1, Q5 BSS138, U2 SIM7000G

Commit message: schematic ready
Parts:
- removed C11: 100nF, symbol Device:C
- added C22: 100nF, symbol Device:C
- added C23, C24, C25: 100µF, symbol Device:C_Polarized
- added C26: 1µF, symbol Device:C
- added D5: PESD3V3L1BSLZ, PESD3V3L1BSL:PESD3V3L1BSLZ, symbol PESD3V3L1BSLZ:PESD3V3L1BSLZ
- added FB1: 280Ω, symbol Device:FerriteBead
- added Q2: BSS138, SOT95P240X120-3N, symbol BSS138:BSS138
- added S2: SLW-1276864-4A-D, SLW-1276864-4A-D:SLW12768644AD, symbol SLW-1276864-4A-D:SLW-1276864-4A-D
- added TP6: TestPoint, symbol Connector:TestPoint
- IC13: footprint SOP65P640X120-20N -> TXB0108PWR:SOP65P640X120-20N
Connections:
- net BAT+: now also S2.2 (COM); no longer U2.P$55 (VBAT@1), U2.P$56 (VBAT@2), U2.P$57 (VBAT@3)
- net GND: now also J6.C4 (SHIELD), J6.C8 (SHIELD), C22.2, C23.2, C24.2, C25.2, C26.2, D5.1 (K1), Q2.2 (S)
- net PWRKEY: now also Q2.1 (G); no longer U2.P$1 (PWRKEY)
- net OUT1.8V: now reaches U2.P$15 (VDD_EXT)
- net OUT1.8V: now also IC13.2 (VCCA), R19.1, TP6.1
- net at U2.P$6 (BOOT_CFG): now also TP2.1
- net NRESET: no longer names the net of U2.P$16 (NRESET)
- new net: C22.1, C23.1, C24.1, C25.1, C26.1, FB1.2, U2.P$55 (VBAT@1), U2.P$56 (VBAT@2), U2.P$57 (VBAT@3)
- new net: Q2.3 (D), U2.P$1 (PWRKEY)
- new net: D5.2 (K2), FB1.1, S2.3 (NO)
- no-connect marks 28 -> 30

Commit message: footprints assigned
Parts:
- C10: footprint CAPC1608X90N -> CL10B104KO8NNNC:CAPC1608X90N
- C12, C13, C26: footprint (none) -> Capacitor_THT:C_Disc_D5.0mm_W2.5mm_P2.50mm
- C22, C23, C24, C25: footprint (none) -> Capacitor_THT:CP_Radial_Tantal_D5.0mm_P2.50mm
- D4: footprint (none) -> Diode_THT:D_DO-41_SOD81_P7.62mm_Horizontal
- FB1: footprint (none) -> Inductor_SMD:L_0805_2012Metric_Pad1.05x1.20mm_HandSolder
- J7: footprint (none) -> Connector_Coaxial:U.FL_Molex_MCRF_73412-0110_Vertical
- Q2, Q5: footprint SOT95P240X120-3N -> BSS138:SOT95P240X120-3N
- R18, R19, R20, R21: footprint (none) -> Resistor_THT:R_Axial_DIN0207_L6.3mm_D2.5mm_P7.62mm_Horizontal
- TP1, TP2, TP3, TP4, TP5, TP6: footprint (none) -> TestPoint:TestPoint_THTPad_D2.0mm_Drill1.0mm
Changed lines of the file:
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@@
 			)
 		)
-		(property "Footprint" ""
+		(property "Footprint" "Connector_Coaxial:U.FL_Molex_MCRF_73412-0110_Vertical"
 			(at 69.85 33.02 0)
 			(effects
@@
 			)
 		)
-		(property "Footprint" ""
+		(property "Footprint" "Capacitor_THT:CP_Radial_Tantal_D5.0mm_P2.50mm"
 			(at 228.2952 48.26 0)
 			(effects
@@
 			)
 		)
-		(property "Footprint" ""
+		(property "Footprint" "TestPoint:TestPoint_THTPad_D2.0mm_Drill1.0mm"
 			(at 86.36 170.18 0)
 			(effects
@@
 			)
 		)
-		(property "Footprint" ""
+		(property "Footprint" "Capacitor_THT:CP_Radial_Tantal_D5.0mm_P2.50mm"
 			(at 256.2352 48.26 0)
 			(effects
@@
 			)
 		)
-		(property "Footprint" ""
+		(property "Footprint" "TestPoint:TestPoint_THTPad_D2.0mm_Drill1.0mm"
 			(at 101.6 170.18 0)
 			(effects
@@
 			)
 		)
-		(property "Footprint" "SOT95P240X120-3N"
+		(property "Footprint" "BSS138:SOT95P240X120-3N"
 			(at 26.67 -44.12 0)
 			(effects
@@
 			)
 		)
-		(property "Footprint" ""
+		(property "Footprint" "TestPoint:TestPoint_THTPad_D2.0mm_Drill1.0mm"
 			(at 15.24 142.24 0)
 			(effects
@@
 			)
 		)
-		(property "Footprint" ""
+		(property "Footprint" "Capacitor_THT:C_Disc_D5.0mm_W2.5mm_P2.50mm"
 			(at 103.8352 26.67 0)
 			(effects
@@
 			)
 		)
-		(property "Footprint" ""
+		(property "Footprint" "Capacitor_THT:C_Disc_D5.0mm_W2.5mm_P2.50mm"
 			(at 216.8652 48.26 0)
 			(effects
@@
 			)
 		)
-		(property "Footprint" ""
+		(property "Footprint" "Resistor_THT:R_Axial_DIN0207_L6.3mm_D2.5mm_P7.62mm_Horizontal"
 			(at 170.942 140.97 90)
 			(effects
@@
 			)
 		)
-		(property "Footprint" ""
+		(property "Footprint" "Resistor_THT:R_Axial_DIN0207_L6.3mm_D2.5mm_P7.62mm_Horizontal"
 			(at 80.01 31.242 90)
 			(effects
@@
 			)
 		)
-		(property "Footprint" ""
+		(property "Footprint" "Inductor_SMD:L_0805_2012Metric_Pad1.05x1.20mm_HandSolder"
 			(at 261.112 29.21 90)
 			(effects
@@
 			)
 		)
-		(property "Footprint" ""
+		(property "Footprint" "Capacitor_THT:CP_Radial_Tantal_D5.0mm_P2.50mm"
 			(at 242.2652 48.26 0)
 			(effects
@@
 			)
 		)
-		(property "Footprint" ""
+		(property "Footprint" "TestPoint:TestPoint_THTPad_D2.0mm_Drill1.0mm"
 			(at 38.1 92.71 0)
 			(effects
@@
 			)
 		)
-		(property "Footprint" ""
+		(property "Footprint" "TestPoint:TestPoint_THTPad_D2.0mm_Drill1.0mm"
 			(at 106.68 177.8 0)
 			(effects
@@
 			)
 		)
-		(property "Footprint" ""
+		(property "Footprint" "Capacitor_THT:CP_Radial_Tantal_D5.0mm_P2.50mm"
 			(at 204.1652 48.26 0)
 			(effects
@@
 			)
 		)
-		(property "Footprint" ""
+		(property "Footprint" "Resistor_THT:R_Axial_DIN0207_L6.3mm_D2.5mm_P7.62mm_Horizontal"
 			(at 160.02 32.512 90)
 			(effects
@@
 			)
 		)
-		(property "Footprint" "SOT95P240X120-3N"
+		(property "Footprint" "BSS138:SOT95P240X120-3N"
 			(at 181.61 144.45 0)
 			(effects
@@
 			)
 		)
-		(property "Footprint" "CAPC1608X90N"
+		(property "Footprint" "CL10B104KO8NNNC:CAPC1608X90N"
 			(at 233.68 182.55 0)
 			(effects
@@
 			)
 		)
-		(property "Footprint" ""
+		(property "Footprint" "Resistor_THT:R_Axial_DIN0207_L6.3mm_D2.5mm_P7.62mm_Horizontal"
 			(at 93.98 31.242 90)
 			(effects
@@
 			)
 		)
-		(property "Footprint" ""
+		(property "Footprint" "Capacitor_THT:C_Disc_D5.0mm_W2.5mm_P2.50mm"
 			(at 87.3252 29.21 0)
 			(effects
@@
 			)
 		)
-		(property "Footprint" ""
+		(property "Footprint" "TestPoint:TestPoint_THTPad_D2.0mm_Drill1.0mm"
 			(at 81.28 176.53 0)
 			(effects
@@
 			)
 		)
-		(property "Footprint" ""
+		(property "Footprint" "Diode_THT:D_DO-41_SOD81_P7.62mm_Horizontal"
 			(at 170.18 34.29 0)
 			(effects

Commit message: updated to hierarchical labels
Parts:
- added S3: SLW-1276864-4A-D, SLW-1276864-4A-D:SLW12768644AD, symbol SLW-1276864-4A-D:SLW-1276864-4A-D
Connections:
- net BAT+: no longer S2.2 (COM)
- net GSM_RXD: now also IC13.1 (A1), IC13.20 (B1); no longer IC13.16 (B4), IC13.4 (A3)
- net GSM_TXD: now also IC13.18 (B2), IC13.3 (A2); no longer IC13.17 (B3), IC13.5 (A4)
- net STATUS: no longer IC13.8 (A7)
- net DCD: no longer names the net of U2.P$5 (DCD)
- net DCD: no longer IC13.7 (A6)
- net DTR: no longer names the net of U2.P$3 (DTR)
- net DTR: no longer IC13.9 (A8)
- removed net GSM_CTS: IC13.1 (A1), IC13.18 (B2), U2.P$7 (CTS)
- net GSM_DCD: no longer names the net of IC13.14 (B6)
- net GSM_DTR: no longer names the net of IC13.12 (B8)
- net GSM_RI: no longer names the net of IC13.15 (B5)
- removed net GSM_RTS: IC13.20 (B1), IC13.3 (A2), U2.P$8 (RTS)
- net GSM_STATUS: no longer names the net of IC13.13 (B7)
- net RI: no longer names the net of U2.P$4 (RI)
- net RI: no longer IC13.6 (A5)
- new net: S2.2 (COM), S3.2 (COM)
- no-connect marks 30 -> 34

Commit message: new footprints assigned
Parts:
- removed IC13: TXB0108PWR, TXB0108PWR:SOP65P640X120-20N, symbol TXB0108PWR:TXB0108PWR
- added IC2: TXB0104PWR, Smartball_footprints:SOP65P640X120-14N, symbol TXB0104PWR:TXB0104PWR
- D5: footprint PESD3V3L1BSL:PESD3V3L1BSLZ -> PESD3V3L1BSLZ:PESD3V3L1BSLZ
Connections:
- net GND: now also IC2.7 (GND)
- net GSM_RXD: now also IC2.13 (B1), IC2.2 (A1)
- net GSM_TXD: now also IC2.12 (B2), IC2.3 (A2)
- net OUT1.8V: now also IC2.1 (VCCA)
- net VOUT_3V3: now also IC2.14 (VCCB)
- net at R19.2: now also IC2.8 (OE)
- no-connect marks 34 -> 40

Commit message: last modifications schematic
Parts:
- removed Q2: BSS138, BSS138:SOT95P240X120-3N, symbol BSS138:BSS138
Connections:
- net OUT+5V: now also S3.3 (NO)
- net PWRKEY: now also IC2.11 (B3), IC2.4 (A3), U2.P$1 (PWRKEY)
- net STATUS: now also IC2.10 (B4), IC2.5 (A4)
- no-connect marks 40 -> 38
