File: PCB/smartBall/Movement.kicad_sch (KiCad schematic)
At the start: 11 parts, among them IC7 ADM7155ACPZ-04-R7, IC9 LSM6DSV16BXTR, J3 QVAR

Commit message: schematic ready
Parts:
- removed C1, C2, C9: CL10B105KO8NNNC, CAPC1608X90N, symbol CL10B105KO8NNNC:CL10B105KO8NNNC
- removed C7: 10µF, symbol Device:C
- added C1, C9: 1µF, symbol Device:C_Polarized
- added C11, C2: 10µF, symbol Device:C_Polarized
- added J9: Conn_01x15, symbol Connector_Generic:Conn_01x15
- AC1: footprint LIS3DHTR -> H3LIS331DLTR:LIS3DHTR
- IC7: footprint SON50P300X300X80-9N-D -> ADM7155ACPZ-04-07:SON50P300X300X80-9N-D
- IC9: footprint LSM6DSV16BXTR -> LSM6DSV16BXTR:LSM6DSV16BXTR
- R14: value 17.5kΩ -> 175kΩ
- R15: value 10kΩ -> 100kΩ
Connections:
- net +3V3: now also C11.1
- net ACCEL_CS: now also J9.4 (Pin_4)
- net ACCEL_INT1: now also J9.3 (Pin_3)
- net ACCEL_INT2: now also J9.2 (Pin_2)
- net BCLK: now also J9.9 (Pin_9)
- net DATA_IN: now also J9.8 (Pin_8)
- net GND: now also C1.2, C11.2, C2.2, C9.2, J9.14 (Pin_14)
- net IMU_CS: now also J9.13 (Pin_13)
- net IMU_INT1: now also J9.10 (Pin_10)
- net IMU_INT2: now also J9.11 (Pin_11)
- net MISO: now also J9.5 (Pin_5)
- net MOSI: now also J9.6 (Pin_6)
- net SCLK: now also J9.7 (Pin_7)
- net VOUT_3V3: now also J9.1 (Pin_1); no longer R14.1
- net at IC7.3 (BYP): now also C9.1
- net at IC7.1 (VREG): now also C2.1
- net at IC7.6 (REF): now also R14.1, C1.1
- net LRCK renamed WCLK
- net WCLK: now also J9.12 (Pin_12)
Other:
- moved on the sheet: R14, R15

Commit message: footprints assigned
Parts:
- C1, C11, C2, C6, C9: footprint (none) -> Capacitor_THT:CP_Radial_Tantal_D5.0mm_P2.50mm
- J3: footprint (none) -> Connector_JST:JST_PH_B3B-PH-K_1x03_P2.00mm_Vertical
- J9: footprint (none) -> Connector_PinHeader_2.54mm:PinHeader_1x15_P2.54mm_Vertical
- R14, R15: footprint (none) -> Resistor_THT:R_Axial_DIN0207_L6.3mm_D2.5mm_P7.62mm_Horizontal
Changed lines of the file:
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@@
 			)
 		)
-		(property "Footprint" ""
+		(property "Footprint" "Resistor_THT:R_Axial_DIN0207_L6.3mm_D2.5mm_P7.62mm_Horizontal"
 			(at 179.832 168.91 90)
 			(effects
@@
 			)
 		)
-		(property "Footprint" ""
+		(property "Footprint" "Resistor_THT:R_Axial_DIN0207_L6.3mm_D2.5mm_P7.62mm_Horizontal"
 			(at 179.832 154.94 90)
 			(effects
@@
 			)
 		)
-		(property "Footprint" ""
+		(property "Footprint" "Connector_PinHeader_2.54mm:PinHeader_1x15_P2.54mm_Vertical"
 			(at 124.46 22.86 0)
 			(effects
@@
 			)
 		)
-		(property "Footprint" ""
+		(property "Footprint" "Capacitor_THT:CP_Radial_Tantal_D5.0mm_P2.50mm"
 			(at 108.9152 157.48 0)
 			(effects
@@
 			)
 		)
-		(property "Footprint" ""
+		(property "Footprint" "Connector_JST:JST_PH_B3B-PH-K_1x03_P2.00mm_Vertical"
 			(at 243.84 88.9 0)
 			(effects
@@
 			)
 		)
-		(property "Footprint" ""
+		(property "Footprint" "Capacitor_THT:CP_Radial_Tantal_D5.0mm_P2.50mm"
 			(at 165.4048 116.84 0)
 			(effects
@@
 			)
 		)
-		(property "Footprint" ""
+		(property "Footprint" "Capacitor_THT:CP_Radial_Tantal_D5.0mm_P2.50mm"
 			(at 122.2248 113.03 0)
 			(effects
@@
 			)
 		)
-		(property "Footprint" ""
+		(property "Footprint" "Capacitor_THT:CP_Radial_Tantal_D5.0mm_P2.50mm"
 			(at 194.31 141.2748 0)
 			(effects
@@
 			)
 		)
-		(property "Footprint" ""
+		(property "Footprint" "Capacitor_THT:CP_Radial_Tantal_D5.0mm_P2.50mm"
 			(at 106.3752 135.89 0)
 			(effects

Commit message: updated to hierarchical labels
Parts:
- removed C1, C9: 1µF, Capacitor_THT:CP_Radial_Tantal_D5.0mm_P2.50mm, symbol Device:C_Polarized
- removed C11, C2: 10µF, Capacitor_THT:CP_Radial_Tantal_D5.0mm_P2.50mm, symbol Device:C_Polarized
- removed C6: 10µF, Capacitor_THT:CP_Radial_Tantal_D5.0mm_P2.50mm, symbol Device:C
- removed IC7: ADM7155ACPZ-04-R7, ADM7155ACPZ-04-07:SON50P300X300X80-9N-D, symbol ADM7155ACPZ-04-R7:ADM7155ACPZ-04-R7
- removed J9: Conn_01x15, Connector_PinHeader_2.54mm:PinHeader_1x15_P2.54mm_Vertical, symbol Connector_Generic:Conn_01x15
- removed R14: 175kΩ, Resistor_THT:R_Axial_DIN0207_L6.3mm_D2.5mm_P7.62mm_Horizontal, symbol Device:R
- removed R15: 100kΩ, Resistor_THT:R_Axial_DIN0207_L6.3mm_D2.5mm_P7.62mm_Horizontal, symbol Device:R
Connections:
- net WCLK: no longer IC9.11 (WCLK)

Commit message: last modifications schematic
Connections:
- net WCLK: now also IC9.11 (WCLK)
Changed lines of the file:
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@@
 	)
 	(hierarchical_label "IMU_INT1"
-		(shape input)
+		(shape output)
 		(at 167.64 77.47 180)
 		(effects
@@
 	)
 	(hierarchical_label "ACCEL_INT2"
-		(shape input)
+		(shape output)
 		(at 106.68 86.36 0)
 		(effects
@@
 	)
 	(hierarchical_label "MISO"
-		(shape input)
+		(shape output)
 		(at 165.1 69.85 180)
 		(effects
@@
 	)
 	(hierarchical_label "IMU_INT2"
-		(shape input)
+		(shape output)
 		(at 215.9 72.39 0)
 		(effects
@@
 	)
 	(hierarchical_label "ACCEL_INT1"
-		(shape input)
+		(shape output)
 		(at 106.68 82.55 0)
 		(effects
@@
 	)
 	(hierarchical_label "MISO"
-		(shape input)
+		(shape output)
 		(at 74.93 120.65 270)
 		(effects
@@
 	)
 	(hierarchical_label "DATA_IN"
-		(shape input)
+		(shape output)
 		(at 154.94 72.39 180)
 		(effects
@@
 	(hierarchical_label "WCLK"
 		(shape input)
-		(at 218.44 69.85 0)
+		(at 217.17 69.85 0)
 		(effects
 			(font
