File: PCB/smartBall/Power.kicad_sch (KiCad schematic)
At the start: 26 parts, among them IC10 BQ51013BRHLR, IC5 MAX17048G+T10, J1 UJ20-C-H-G-MSMT-R-4C-P16-TR, U1 MCP73871-2CA

Commit message: schematic ready
Parts:
- removed L1: L, symbol Device:L
- added C27, C7: 4.7µF, symbol Device:C
- added C28, C30, C31, C32, C33: 10µF, symbol Device:C
- added C29: 0.1µF, symbol Device:C_Polarized
- added C34: 0.47µF, symbol Device:C
- added C35: 20µF, symbol Device:C
- added C36: 1µF, symbol Device:C
- added C37: C, symbol Device:C
- added D6: LED, symbol Device:LED
- added J8: Conn_01x02, symbol Connector_Generic:Conn_01x02
- added Q6: Si2323DDS-T1-GE3, Si2323DDS-T1-GE3:SOT95P237X112-3N, symbol Si2323DDS-T1-GE3:Si2323DDS-T1-GE3
- added R27: 470Ω, symbol Device:R
- added TH1, TH2: 10kΩ, symbol Device:Thermistor_NTC
- C3: value 10nF -> 0.47µF
- C4: value 10nF -> C
- C5: value 10µF/10V -> 10µF
- D1, D2: footprint DIOM5227X270N -> SS14:DIOM5227X270N
- IC10: footprint BQ51050BRHLR -> BQ51013BRHLR:BQ51050BRHLR
- IC5: footprint SON50P200X200X80-9N-D -> MAX17048G+T10:SON50P200X200X80-9N-D
- J1: footprint UJ20CHGMSMTR4CP16TR -> UJ20-C-H-G-MSMT-R-4C-P16-TR:UJ20CHGMSMTR4CP16TR
- R1: value 10kΩ -> 1.5kΩ
- R10: value R -> 200Ω
- R13: value R -> 20kΩ
- R2: value 1kΩ -> 10kΩ
- R24, R25: value 10kΩ -> 470Ω
- R9: value 10kΩ -> 66Ω
- S1: footprint SLW12768644AD -> SLW-1276864-4A-D:SLW12768644AD
Connections:
- net VOUT_3V3 is gone; now on net CHARGER_SRC: R24.2, R25.2
- net BAT+: now also C27.2, C29.1
- net GND: now also D3.2 (GND), IC10.1 (PGND_1), IC10.10 (EN1), IC10.11 (EN2), IC10.20 (PGND_2), IC10.21 (EP), C27.1, C28.1, C29.2, C35.2, C36.2, C7.2, TH1.2; no longer C5.1, IC10.8 (~{AD-EN}), IC10.9 (AD), R1.2, R13.1, R9.2
- net USB_D+: now also D3.1 (I/O1_1), D3.6 (I/O1_2)
- net USB_D-: now also D3.3 (I/O2_1), D3.4 (I/O2_2)
- net at IC10.14 (FOD): now also R10.2, R13.1, R9.1; no longer R13.2
- net at D2.2 (A), J1.A4 (VBUS_1), J1.A9 (VBUS_2): now also D3.5 (VBUS), Q6.2 (S); no longer C5.2, IC10.18 (RECT)
- net at C4.1: now also C3.1, IC10.19 (AC2), C32.1, C33.1, J8.2 (Pin_2)
- net at C3.2: now also IC10.16 (CLAMP2)
- net CHARGER_SRC: now reaches D1.1 (K), U1.18 (IN), U1.19 (IN), U1.2 (VPCC), U1.3 (SEL)
- net CHARGER_SRC: now also U1.17 (CE), U1.4 (PROG2), C28.2, Q6.3 (D), R27.1; no longer D2.1 (K)
- net at U1.5 (THERM): now also TH1.1; no longer R1.1
- net at S1.2 (COM), U1.1 (OUT), U1.20 (OUT): now also C7.1
- net at IC10.12 (ILIM): now also R9.2; no longer R10.2
- net at IC10.13 (TS/CTRL): now also TH2.2; no longer R9.1
- net at IC10.15 (COMM2): now also C33.2
- net at IC10.17 (BOOT2): now also C32.2
- net at IC10.2 (AC1): now also C30.2, C31.2, C34.2, C37.2; no longer C4.2
- net at IC10.3 (BOOT1): now also IC10.5 (CLAMP1), IC10.8 (~{AD-EN}), C30.1, C34.1, Q6.1 (G)
- net at IC10.4 (OUT): now also C5.1; no longer D1.2 (A)
- net at IC10.6 (COMM1): now also C31.1
- net at IC10.7 (~{CHG}): now also R1.1
- net ~PG: no longer names the net of U1.6 (~{PG})
- net ~PG: now also R27.2
- new net: C35.1, IC10.18 (RECT), R13.2
- new net: C37.1, C4.2, J8.1 (Pin_1)
- new net: D6.1 (K), R1.2
- new net: C5.2, D1.2 (A), D6.2 (A)
- new net USB_SRC: C36.1, D2.1 (K), IC10.9 (AD)
- no-connect marks 0 -> 2
Other:
- moved on the sheet: D1, D2, D3, IC10

Commit message: footprints assigned
Parts:
- BT1: footprint (none) -> Connector_Wire:SolderWire-0.75sqmm_1x02_P4.8mm_D1.25mm_OD2.3mm
- C27, C28, C29, C3, C30, C31, C32, C33, C34, C35, C36, C37, C4, C5, C7: footprint (none) -> Capacitor_THT:CP_Radial_Tantal_D5.0mm_P2.50mm
- D6: footprint (none) -> Diode_THT:D_DO-41_SOD81_P7.62mm_Horizontal
- J8: footprint (none) -> Connector_PinHeader_2.54mm:PinHeader_1x02_P2.54mm_Vertical
- R1, R10, R11, R12, R13, R2, R24, R25, R27, R5, R6, R7, R8, R9, TH1, TH2: footprint (none) -> Resistor_THT:R_Axial_DIN0207_L6.3mm_D2.5mm_P7.62mm_Horizontal
Changed lines of the file:
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@@
 			)
 		)
-		(property "Footprint" ""
+		(property "Footprint" "Capacitor_THT:CP_Radial_Tantal_D5.0mm_P2.50mm"
 			(at 35.56 64.4652 0)
 			(effects
@@
 			)
 		)
-		(property "Footprint" ""
+		(property "Footprint" "Capacitor_THT:CP_Radial_Tantal_D5.0mm_P2.50mm"
 			(at 92.71 72.0852 0)
 			(effects
@@
 			)
 		)
-		(property "Footprint" ""
+		(property "Footprint" "Capacitor_THT:CP_Radial_Tantal_D5.0mm_P2.50mm"
 			(at 150.8252 156.21 0)
 			(effects
@@
 			)
 		)
-		(property "Footprint" ""
+		(property "Footprint" "Resistor_THT:R_Axial_DIN0207_L6.3mm_D2.5mm_P7.62mm_Horizontal"
 			(at 191.262 123.19 90)
 			(effects
@@
 			)
 		)
-		(property "Footprint" ""
+		(property "Footprint" "Capacitor_THT:CP_Radial_Tantal_D5.0mm_P2.50mm"
 			(at 53.0352 119.38 0)
 			(effects
@@
 			)
 		)
-		(property "Footprint" ""
+		(property "Footprint" "Resistor_THT:R_Axial_DIN0207_L6.3mm_D2.5mm_P7.62mm_Horizontal"
 			(at 106.68 71.882 90)
 			(effects
@@
 			)
 		)
-		(property "Footprint" ""
+		(property "Footprint" "Resistor_THT:R_Axial_DIN0207_L6.3mm_D2.5mm_P7.62mm_Horizontal"
 			(at 234.442 30.48 90)
 			(effects
@@
 			)
 		)
-		(property "Footprint" ""
+		(property "Footprint" "Capacitor_THT:CP_Radial_Tantal_D5.0mm_P2.50mm"
 			(at 90.17 67.0052 0)
 			(effects
@@
 			)
 		)
-		(property "Footprint" ""
+		(property "Footprint" "Resistor_THT:R_Axial_DIN0207_L6.3mm_D2.5mm_P7.62mm_Horizontal"
 			(at 45.72 161.29 0)
 			(effects
@@
 			)
 		)
-		(property "Footprint" ""
+		(property "Footprint" "Capacitor_THT:CP_Radial_Tantal_D5.0mm_P2.50mm"
 			(at 27.6352 57.15 0)
 			(effects
@@
 			)
 		)
-		(property "Footprint" ""
+		(property "Footprint" "Resistor_THT:R_Axial_DIN0207_L6.3mm_D2.5mm_P7.62mm_Horizontal"
 			(at 24.892 149.86 90)
 			(effects
@@
 			)
 		)
-		(property "Footprint" ""
+		(property "Footprint" "Connector_PinHeader_2.54mm:PinHeader_1x02_P2.54mm_Vertical"
 			(at 46.99 30.48 0)
 			(effects
@@
 			)
 		)
-		(property "Footprint" ""
+		(property "Footprint" "Capacitor_THT:CP_Radial_Tantal_D5.0mm_P2.50mm"
 			(at 112.7252 139.7 0)
 			(effects
@@
 			)
 		)
-		(property "Footprint" ""
+		(property "Footprint" "Resistor_THT:R_Axial_DIN0207_L6.3mm_D2.5mm_P7.62mm_Horizontal"
 			(at 221.742 146.05 90)
 			(effects
@@
 			)
 		)
-		(property "Footprint" ""
+		(property "Footprint" "Resistor_THT:R_Axial_DIN0207_L6.3mm_D2.5mm_P7.62mm_Horizontal"
 			(at 87.63 56.642 90)
 			(effects
@@
 			)
 		)
-		(property "Footprint" ""
+		(property "Footprint" "Capacitor_THT:CP_Radial_Tantal_D5.0mm_P2.50mm"
 			(at 98.7552 134.62 0)
 			(effects
@@
 			)
 		)
-		(property "Footprint" ""
+		(property "Footprint" "Capacitor_THT:CP_Radial_Tantal_D5.0mm_P2.50mm"
 			(at 35.2552 90.17 0)
 			(effects
@@
 			)
 		)
-		(property "Footprint" ""
+		(property "Footprint" "Resistor_THT:R_Axial_DIN0207_L6.3mm_D2.5mm_P7.62mm_Horizontal"
 			(at 106.68 61.722 90)
 			(effects
@@
 			)
 		)
-		(property "Footprint" ""
+		(property "Footprint" "Connector_Wire:SolderWire-0.75sqmm_1x02_P4.8mm_D1.25mm_OD2.3mm"
 			(at 123.19 155.956 90)
 			(effects
@@
 			)
 		)
-		(property "Footprint" ""
+		(property "Footprint" "Capacitor_THT:CP_Radial_Tantal_D5.0mm_P2.50mm"
 			(at 92.4052 88.9 0)
 			(effects
@@
 			)
 		)
-		(property "Footprint" ""
+		(property "Footprint" "Resistor_THT:R_Axial_DIN0207_L6.3mm_D2.5mm_P7.62mm_Horizontal"
 			(at 29.21 73.152 90)
 			(effects
@@
 			)
 		)
-		(property "Footprint" ""
+		(property "Footprint" "Resistor_THT:R_Axial_DIN0207_L6.3mm_D2.5mm_P7.62mm_Horizontal"
 			(at 158.242 41.91 90)
 			(effects
@@
 			)
 		)
-		(property "Footprint" ""
+		(property "Footprint" "Capacitor_THT:CP_Radial_Tantal_D5.0mm_P2.50mm"
 			(at 18.7452 78.74 0)
 			(effects
@@
 			)
 		)
-		(property "Footprint" ""
+		(property "Footprint" "Resistor_THT:R_Axial_DIN0207_L6.3mm_D2.5mm_P7.62mm_Horizontal"
 			(at 210.312 135.89 90)
 			(effects
@@
 			)
 		)
-		(property "Footprint" ""
+		(property "Footprint" "Resistor_THT:R_Axial_DIN0207_L6.3mm_D2.5mm_P7.62mm_Horizontal"
 			(at 90.932 167.64 90)
 			(effects
@@
 			)
 		)
-		(property "Footprint" ""
+		(property "Footprint" "Resistor_THT:R_Axial_DIN0207_L6.3mm_D2.5mm_P7.62mm_Horizontal"
 			(at 101.092 171.45 90)
 			(effects
@@
 			)
 		)
-		(property "Footprint" ""
+		(property "Footprint" "Capacitor_THT:CP_Radial_Tantal_D5.0mm_P2.50mm"
 			(at 60.96 46.6852 0)
 			(effects
@@
 			)
 		)
-		(property "Footprint" ""
+		(property "Footprint" "Capacitor_THT:CP_Radial_Tantal_D5.0mm_P2.50mm"
 			(at 35.56 69.5452 0)
 			(effects
@@
 			)
 		)
-		(property "Footprint" ""
+		(property "Footprint" "Diode_THT:D_DO-41_SOD81_P7.62mm_Horizontal"
 			(at 24.13 81.28 0)
 			(effects
@@
 			)
 		)
-		(property "Footprint" ""
+		(property "Footprint" "Capacitor_THT:CP_Radial_Tantal_D5.0mm_P2.50mm"
 			(at 85.09 69.5452 0)
 			(effects
@@
 			)
 		)
-		(property "Footprint" ""
+		(property "Footprint" "Resistor_THT:R_Axial_DIN0207_L6.3mm_D2.5mm_P7.62mm_Horizontal"
 			(at 113.03 48.26 0)
 			(effects
@@
 			)
 		)
-		(property "Footprint" ""
+		(property "Footprint" "Capacitor_THT:CP_Radial_Tantal_D5.0mm_P2.50mm"
 			(at 29.21 72.0852 0)
 			(effects
@@
 			)
 		)
-		(property "Footprint" ""
+		(property "Footprint" "Resistor_THT:R_Axial_DIN0207_L6.3mm_D2.5mm_P7.62mm_Horizontal"
 			(at 29.972 158.75 90)
 			(effects
@@
 			)
 		)
-		(property "Footprint" ""
+		(property "Footprint" "Resistor_THT:R_Axial_DIN0207_L6.3mm_D2.5mm_P7.62mm_Horizontal"
 			(at 96.52 151.892 90)
 			(effects

Commit message: updated to hierarchical labels
Parts:
- added J11, J12: Conn_01x15, Connector_PinHeader_2.54mm:PinHeader_1x15_P2.54mm_Vertical, symbol Connector_Generic:Conn_01x15
- D3: DESCRIPTION Low Cap. ESD Protection Auto SOT-23-6 STMicroelectronics US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 -> (none)
Connections:
- net BAT+: now also J11.12 (Pin_12)
- net FG_ALRT: now also J11.9 (Pin_9)
- net I2C_SCL: now also J11.10 (Pin_10)
- net I2C_SDA: now also J11.11 (Pin_11)
- net STAT1: now also J11.7 (Pin_7)
- net STAT2: now also J11.8 (Pin_8)
- net USB_D+: now also J11.5 (Pin_5)
- net USB_D-: now also J11.6 (Pin_6)
- net +3V3 renamed Movement/VOUT_3V3
- net Movement/VOUT_3V3: now also J11.1 (Pin_1)
- new net Movement/ACCEL_CS: J12.1 (Pin_1)
- new net Movement/ACCEL_INT1: J12.2 (Pin_2)
- new net Movement/ACCEL_INT2: J12.3 (Pin_3)
- new net Movement/BCLK: J12.4 (Pin_4)
- new net Movement/DATA_IN: J12.5 (Pin_5)
- new net Movement/IMU_CS: J12.6 (Pin_6)
- new net Movement/IMU_INT1: J12.7 (Pin_7)
- new net Movement/IMU_INT2: J12.8 (Pin_8)
- new net Movement/MISO: J12.9 (Pin_9)
- new net Movement/MOSI: J12.10 (Pin_10)
- new net Movement/SCLK: J12.11 (Pin_11)
- new net Movement/WCLK: J12.12 (Pin_12)
- new net STEP_UP/LOUDNESS: J11.4 (Pin_4)
- new net STEP_UP/OUT+5V: J11.3 (Pin_3)
- no-connect marks 2 -> 3
Other:
- added sheet Movement (Movement.kicad_sch)
- sheet STEP_UP ports: added +3V3, LOUDNESS, OUT+5V, V_SYS; removed none

Commit message: last modifications schematic
Connections:
- net GND: now also IC5.9 (EP), TH2.1
- net TS/CTRL: now reaches IC10.13 (TS/CTRL), TH2.2
- net TS/CTRL: now also J11.2 (Pin_2)
- no-connect marks 3 -> 8
Changed lines of the file:
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@@
 	)
 	(junction
+		(at 113.03 60.96)
+		(diameter 0)
+		(color 0 0 0 0)
+	)
+	(junction
 		(at 102.87 161.29)
 		(diameter 0)
@@
 	)
 	(junction
+		(at 203.2 144.78)
+		(diameter 0)
+		(color 0 0 0 0)
+	)
+	(junction
 		(at 97.79 175.26)
 		(diameter 0)
@@
 	)
 	(no_connect
+		(at 251.46 138.43)
+	)
+	(no_connect
+		(at 251.46 140.97)
+	)
+	(no_connect
+		(at 281.94 38.1)
+	)
+	(no_connect
+		(at 251.46 135.89)
+	)
+	(no_connect
+		(at 279.4 38.1)
+	)
+	(no_connect
 		(at 222.25 38.1)
 	)
 	(no_connect
-		(at 251.46 107.95)
+		(at 284.48 38.1)
 	)
 	(wire
@@
 	(wire
 		(pts
+			(xy 203.2 144.78) (xy 203.2 146.05)
+		)
+		(stroke
+			(width 0)
+			(type default)
+		)
+	)
+	(wire
+		(pts
 			(xy 43.18 68.58) (xy 43.18 63.5)
 		)
@@
 	(wire
 		(pts
+			(xy 199.39 144.78) (xy 203.2 144.78)
+		)
+		(stroke
+			(width 0)
+			(type default)
+		)
+	)
+	(wire
+		(pts
 			(xy 254 54.61) (xy 259.08 54.61)
 		)
@@
 	(wire
 		(pts
+			(xy 113.03 60.96) (xy 118.11 60.96)
+		)
+		(stroke
+			(width 0)
+			(type default)
+		)
+	)
+	(wire
+		(pts
 			(xy 154.94 33.02) (xy 191.77 33.02)
 		)
@@
 	(wire
 		(pts
+			(xy 123.19 46.99) (xy 123.19 43.18)
+		)
+		(stroke
+			(width 0)
+			(type default)
+		)
+	)
+	(wire
+		(pts
 			(xy 48.26 163.83) (xy 48.26 146.05)
 		)
@@
 	(wire
 		(pts
+			(xy 175.26 160.02) (xy 199.39 160.02)
+		)
+		(stroke
+			(width 0)
+			(type default)
+		)
+	)
+	(wire
+		(pts
 			(xy 97.79 175.26) (xy 97.79 177.8)
 		)
@@
 	(wire
 		(pts
+			(xy 175.26 157.48) (xy 175.26 160.02)
+		)
+		(stroke
+			(width 0)
+			(type default)
+		)
+	)
+	(wire
+		(pts
 			(xy 149.86 142.24) (xy 149.86 148.59)
 		)
@@
 	(wire
 		(pts
+			(xy 199.39 160.02) (xy 199.39 144.78)
+		)
+		(stroke
+			(width 0)
+			(type default)
+		)
+	)
+	(wire
+		(pts
 			(xy 248.92 57.15) (xy 248.92 38.1)
 		)
@@
 	(wire
 		(pts
+			(xy 123.19 43.18) (xy 113.03 43.18)
+		)
+		(stroke
+			(width 0)
+			(type default)
+		)
+	)
+	(wire
+		(pts
 			(xy 68.58 15.24) (xy 68.58 13.97)
 		)
@@
 	(wire
 		(pts
+			(xy 113.03 43.18) (xy 113.03 45.72)
+		)
+		(stroke
+			(width 0)
+			(type default)
+		)
+	)
+	(wire
+		(pts
 			(xy 264.16 52.07) (xy 264.16 59.69)
 		)
@@
 	(wire
 		(pts
-			(xy 203.2 142.24) (xy 203.2 146.05)
+			(xy 203.2 142.24) (xy 203.2 144.78)
 		)
 		(stroke
@@
 		)
 	)
+	(label "TS{slash}CTRL"
+		(at 118.11 60.96 0)
+		(effects
+			(font
+				(size 1.27 1.27)
+			)
+			(justify left bottom)
+		)
+	)
+	(label "TS{slash}CTRL"
+		(at 251.46 107.95 180)
+		(effects
+			(font
+				(size 1.27 1.27)
+			)
+			(justify right bottom)
+		)
+	)
 	(label "USB_D+"
 		(at 171.45 38.1 180)
@@
 	(symbol
 		(lib_id "power:GND")
-		(at 129.54 48.26 0)
-		(unit 1)
-		(body_style 1)
-		(exclude_from_sim no)
-		(in_bom yes)
-		(on_board yes)
-		(in_pos_files yes)
-		(dnp no)
-		(fields_autoplaced yes)
-		(property "Reference" "#PWR017"
-			(at 129.54 54.61 0)
-			(hide yes)
-			(show_name no)
-			(do_not_autoplace no)
-			(effects
-				(font
-					(size 1.27 1.27)
-				)
-			)
-		)
-		(property "Value" "GND"
-			(at 129.54 53.34 0)
-			(show_name no)
-			(do_not_autoplace no)
-			(effects
-				(font
-					(size 1.27 1.27)
-				)
-			)
-		)
-		(property "Footprint" ""
-			(at 129.54 48.26 0)
-			(hide yes)
-			(show_name no)
-			(do_not_autoplace no)
-			(effects
-				(font
-					(size 1.27 1.27)
-				)
-			)
-		)
-		(property "Datasheet" ""
-			(at 129.54 48.26 0)
-			(hide yes)
-			(show_name no)
-			(do_not_autoplace no)
-			(effects
-				(font
-					(size 1.27 1.27)
-				)
-			)
-		)
-		(property "Description" "Power symbol creates a global label with name \"GND\" , ground"
-			(at 129.54 48.26 0)
-			(hide yes)
-			(show_name no)
-			(do_not_autoplace no)
-			(effects
-				(font
-					(size 1.27 1.27)
-				)
-			)
-		)
-		(pin "1"
-		)
-		(instances
-			(project "smartBall"
-				(path "/88604d25-498a-4a0c-bf5d-b8ab9ca45bd7/2520541d-587b-4ff4-8d41-f776640f2402"
-					(reference "#PWR017")
-					(unit 1)
-				)
-			)
-		)
-	)
-	(symbol
-		(lib_id "power:GND")
 		(at 191.77 54.61 0)
 		(unit 1)
@@
 	)
 	(symbol
+		(lib_id "power:GND")
+		(at 123.19 46.99 0)
+		(unit 1)
+		(body_style 1)
+		(exclude_from_sim no)
+		(in_bom yes)
+		(on_board yes)
+		(in_pos_files yes)
+		(dnp no)
+		(fields_autoplaced yes)
+		(property "Reference" "#PWR017"
+			(at 123.19 53.34 0)
+			(hide yes)
+			(show_name no)
+			(do_not_autoplace no)
+			(effects
+				(font
+					(size 1.27 1.27)
+				)
+			)
+		)
+		(property "Value" "GND"
+			(at 123.19 52.07 0)
+			(show_name no)
+			(do_not_autoplace no)
+			(effects
+				(font
+					(size 1.27 1.27)
+				)
+			)
+		)
+		(property "Footprint" ""
+			(at 123.19 46.99 0)
+			(hide yes)
+			(show_name no)
+			(do_not_autoplace no)
+			(effects
+				(font
+					(size 1.27 1.27)
+				)
+			)
+		)
+		(property "Datasheet" ""
+			(at 123.19 46.99 0)
+			(hide yes)
+			(show_name no)
+			(do_not_autoplace no)
+			(effects
+				(font
+					(size 1.27 1.27)
+				)
+			)
+		)
+		(property "Description" "Power symbol creates a global label with name \"GND\" , ground"
+			(at 123.19 46.99 0)
+			(hide yes)
+			(show_name no)
+			(do_not_autoplace no)
+			(effects
+				(font
+					(size 1.27 1.27)
+				)
+			)
+		)
+		(pin "1"
+		)
+		(instances
+			(project "smartBall"
+				(path "/88604d25-498a-4a0c-bf5d-b8ab9ca45bd7/2520541d-587b-4ff4-8d41-f776640f2402"
+					(reference "#PWR017")
+					(unit 1)
+				)
+			)
+		)
+	)
+	(symbol
 		(lib_id "Connector_Generic:Conn_01x15")
 		(at 256.54 123.19 0)
@@
 			)
 		)
-		(pin "ACCEL_INT1" input
+		(pin "ACCEL_INT1" output
 			(at 256.54 59.69 90)
 			(effects
@@
 			)
 		)
-		(pin "ACCEL_INT2" input
+		(pin "ACCEL_INT2" output
 			(at 259.08 59.69 90)
 			(effects
@@
 			)
 		)
-		(pin "DATA_IN" input
+		(pin "DATA_IN" output
 			(at 264.16 59.69 90)
 			(effects
@@
 			)
 		)
-		(pin "IMU_INT1" input
+		(pin "IMU_INT1" output
 			(at 269.24 59.69 90)
 			(effects
@@
 			)
 		)
-		(pin "IMU_INT2" input
+		(pin "IMU_INT2" output
 			(at 271.78 59.69 90)
 			(effects
@@
 			)
 		)
-		(pin "MISO" input
+		(pin "MISO" output
 			(at 274.32 59.69 90)
 			(effects
@@
 			)
 		)
-		(pin "OUT+5V" input
+		(pin "OUT+5V" output
 			(at 228.6 92.71 270)
 			(effects
@@
 			)
 		)
-		(pin "+3V3" input
+		(pin "+3V3" output
 			(at 233.68 92.71 270)
 			(effects
