File: PCB/smartBall/Stationary.kicad_sch (KiCad schematic)
At the start: 11 parts, among them IC1 NEO-F10N-00B, IC6 4259-63, IC8 MAX98357AETE+T, J2 Speaker, J4 FXP612 (u.FL) 2, J5 FXP612 (u.FL) 1, Q3 Si2323DDS-T1-GE3, Q4 BSS138

Commit message: schematic ready
Parts:
- added R26: 100kΩ, symbol Device:R
- added R28: 10kΩ, symbol Device:R
- IC6: footprint SOT65P210X110-6N -> 4259-63:SOT65P210X110-6N
- IC8: footprint QFN50P300X300X80-17N -> MAX98357AETE+T:QFN50P300X300X80-17N
- Q3: footprint SOT95P237X112-3N -> Si2323DDS-T1-GE3:SOT95P237X112-3N
- R16: value 330kΩ -> 680kΩ
Connections:
- net VOUT_3V3: no longer IC6.6 (~{CTRL_OR_VDD})
- net at IC1.23 (VCC), Q3.3 (D): now also IC6.6 (~{CTRL_OR_VDD}), R28.1
- net at IC8.2 (GAIN_SLOT): now also R26.1; no longer Q4.3 (D)
- net GPS_EN: no longer names the net of IC1.14 (LNA_EN)
- net RESET_N: no longer names the net of IC1.8 (RESET_N)
- net RESET_N: now also R28.2
- new net: Q4.3 (D), R26.2
- no-connect marks 6 -> 7
Changed lines of the file:
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@@
+	)
+	(junction
+		(at 54.61 87.63)
+		(diameter 0)
+		(color 0 0 0 0)
 	)
 	(junction
@@
 	)
 	(junction
+		(at 119.38 60.96)
+		(diameter 0)
+		(color 0 0 0 0)
+	)
+	(junction
 		(at 15.24 62.23)
 		(diameter 0)
@@
 	)
 	(no_connect
+		(at 39.37 36.83)
+	)
+	(no_connect
 		(at 233.68 88.9)
 	)
@@
 	(wire
 		(pts
+			(xy 200.66 77.47) (xy 200.66 82.55)
+		)
+		(stroke
+			(width 0)
+			(type default)
+		)
+	)
+	(wire
+		(pts
 			(xy 82.55 52.07) (xy 110.49 52.07)
 		)
@@
 	(wire
 		(pts
-			(xy 31.75 36.83) (xy 39.37 36.83)
-		)
-		(stroke
-			(width 0)
-			(type default)
-		)
-	)
-	(wire
-		(pts
-			(xy 82.55 44.45) (xy 87.63 44.45)
+			(xy 82.55 44.45) (xy 91.44 44.45)
 		)
 		(stroke
@@
 	(wire
 		(pts
+			(xy 119.38 60.96) (xy 119.38 87.63)
+		)
+		(stroke
+			(width 0)
+			(type default)
+		)
+	)
+	(wire
+		(pts
 			(xy 134.62 109.22) (xy 127 109.22)
 		)
@@
 	(wire
 		(pts
+			(xy 119.38 87.63) (xy 54.61 87.63)
+		)
+		(stroke
+			(width 0)
+			(type default)
+		)
+	)
+	(wire
+		(pts
 			(xy 15.24 39.37) (xy 39.37 39.37)
 		)
@@
 	(wire
 		(pts
+			(xy 99.06 44.45) (xy 119.38 44.45)
+		)
+		(stroke
+			(width 0)
+			(type default)
+		)
+	)
+	(wire
+		(pts
+			(xy 179.07 72.39) (xy 179.07 60.96)
+		)
+		(stroke
+			(width 0)
+			(type default)
+		)
+	)
+	(wire
+		(pts
 			(xy 15.24 62.23) (xy 39.37 62.23)
 		)
@@
 	(wire
 		(pts
+			(xy 119.38 44.45) (xy 119.38 60.96)
+		)
+		(stroke
+			(width 0)
+			(type default)
+		)
+	)
+	(wire
+		(pts
 			(xy 260.35 91.44) (xy 260.35 71.12)
 		)
@@
 	(wire
 		(pts
+			(xy 200.66 66.04) (xy 200.66 69.85)
+		)
+		(stroke
+			(width 0)
+			(type default)
+		)
+	)
+	(wire
+		(pts
 			(xy 82.55 59.69) (xy 110.49 59.69)
 		)
@@
 	(wire
 		(pts
+			(xy 179.07 60.96) (xy 119.38 60.96)
+		)
+		(stroke
+			(width 0)
+			(type default)
+		)
+	)
+	(wire
+		(pts
 			(xy 127 74.93) (xy 134.62 74.93)
 		)
@@
 		(pts
 			(xy 82.55 57.15) (xy 92.71 57.15)
-		)
-		(stroke
-			(width 0)
-			(type default)
-		)
-	)
-	(wire
-		(pts
-			(xy 200.66 66.04) (xy 200.66 82.55)
 		)
 		(stroke
@@
 		)
 	)
-	(global_label "RESET_N"
+	(global_label "GPS_POWER"
 		(shape bidirectional)
-		(at 87.63 44.45 0)
+		(at 27.94 101.6 180)
 		(fields_autoplaced yes)
 		(effects
@@
 				(size 1.27 1.27)
 			)
-			(justify left)
+			(justify right)
 		)
 		(property "Intersheetrefs" "${INTERSHEET_REFS}"
-			(at 99.7697 44.45 0)
-			(effects
-				(font
-					(size 1.27 1.27)
-				)
-				(justify left)
-				(hide yes)
-			)
-		)
-	)
-	(global_label "GPS_POWER"
+			(at 12.6555 101.6 0)
+			(effects
+				(font
+					(size 1.27 1.27)
+				)
+				(justify right)
+				(hide yes)
+			)
+		)
+	)
+	(global_label "TXD"
 		(shape bidirectional)
-		(at 27.94 101.6 180)
+		(at 31.75 52.07 180)
 		(fields_autoplaced yes)
 		(effects
@@
 		)
 		(property "Intersheetrefs" "${INTERSHEET_REFS}"
-			(at 12.6555 101.6 0)
+			(at 24.2064 52.07 0)
 			(effects
 				(font
@@
 		)
 	)
-	(global_label "GPS_EN"
-		(shape bidirectional)
-		(at 31.75 36.83 180)
+	(global_label "G_BCLK"
+		(shape output)
+		(at 236.22 29.21 90)
 		(fields_autoplaced yes)
 		(effects
@@
 				(size 1.27 1.27)
 			)
-			(justify right)
-		)
-		(property "Intersheetrefs" "${INTERSHEET_REFS}"
-			(at 20.4569 36.83 0)
-			(effects
-				(font
-					(size 1.27 1.27)
-				)
-				(justify right)
-				(hide yes)
-			)
-		)
-	)
-	(global_label "TXD"
-		(shape bidirectional)
-		(at 31.75 52.07 180)
-		(fields_autoplaced yes)
-		(effects
-			(font
-				(size 1.27 1.27)
-			)
-			(justify right)
-		)
-		(property "Intersheetrefs" "${INTERSHEET_REFS}"
-			(at 24.2064 52.07 0)
-			(effects
-				(font
-					(size 1.27 1.27)
-				)
-				(justify right)
-				(hide yes)
-			)
-		)
-	)
-	(global_label "G_BCLK"
-		(shape output)
-		(at 236.22 29.21 90)
-		(fields_autoplaced yes)
-		(effects
-			(font
-				(size 1.27 1.27)
-			)
 			(justify left)
 		)
 		(property "Intersheetrefs" "${INTERSHEET_REFS}"
 			(at 236.22 19.1491 90)
-			(effects
-				(font
-					(size 1.27 1.27)
-				)
-				(justify left)
-				(hide yes)
-			)
-		)
-	)
-	(global_label "VOUT_3V3"
-		(shape bidirectional)
-		(at 179.07 72.39 0)
-		(fields_autoplaced yes)
-		(effects
-			(font
-				(size 1.27 1.27)
-			)
-			(justify left)
-		)
-		(property "Intersheetrefs" "${INTERSHEET_REFS}"
-			(at 192.3589 72.39 0)
 			(effects
 				(font
@@
 			)
 		)
-		(property "Value" "330kΩ"
+		(property "Value" "680kΩ"
 			(at 219.71 87.6299 0)
 			(effects
@@
 			)
 		)
-		(property "Footprint" "SOT95P237X112-3N"
+		(property "Footprint" "Si2323DDS-T1-GE3:SOT95P237X112-3N"
 			(at 58.42 200.33 0)
 			(effects
@@
 			)
 		)
-		(property "Footprint" "QFN50P300X300X80-17N"
+		(property "Footprint" "MAX98357AETE+T:QFN50P300X300X80-17N"
 			(at 255.27 140.64 0)
 			(effects
@@
 			)
 		)
-		(property "Footprint" "SOT65P210X110-6N"
+		(property "Footprint" "4259-63:SOT65P210X110-6N"
 			(at 168.91 167.31 0)
 			(effects
@@
 	)
 	(symbol
+		(lib_id "Device:R")
+		(at 95.25 44.45 270)
+		(unit 1)
+		(exclude_from_sim no)
+		(in_bom yes)
+		(on_board yes)
+		(dnp no)
+		(fields_autoplaced yes)
+		(property "Reference" "R28"
+			(at 95.25 38.1 90)
+			(effects
+				(font
+					(size 1.27 1.27)
+				)
+			)
+		)
+		(property "Value" "10kΩ"
+			(at 95.25 40.64 90)
+			(effects
+				(font
+					(size 1.27 1.27)
+				)
+			)
+		)
+		(property "Footprint" ""
+			(at 95.25 42.672 90)
+			(effects
+				(font
+					(size 1.27 1.27)
+				)
+				(hide yes)
+			)
+		)
+		(property "Datasheet" "~"
+			(at 95.25 44.45 0)
+			(effects
+				(font
+					(size 1.27 1.27)
+				)
+				(hide yes)
+			)
+		)
+		(property "Description" "Resistor"
+			(at 95.25 44.45 0)
+			(effects
+				(font
+					(size 1.27 1.27)
+				)
+				(hide yes)
+			)
+		)
+		(pin "2"
+		)
+		(pin "1"
+		)
+		(instances
+			(project ""
+				(path "/88604d25-498a-4a0c-bf5d-b8ab9ca45bd7/fa45934c-4794-4ba6-bd1a-84173322bb33"
+					(reference "R28")
+					(unit 1)
+				)
+			)
+		)
+	)
+	(symbol
 		(lib_id "BSS138:BSS138")
 		(at 193.04 92.71 0)
@@
 					(unit 1)
 				)
+			)
+		)
+	)
+	(symbol
+		(lib_id "Device:R")
+		(at 200.66 73.66 0)
+		(unit 1)
+		(exclude_from_sim no)
+		(in_bom yes)
+		(on_board yes)
+		(dnp no)
+		(fields_autoplaced yes)
+		(property "Reference" "R26"
+			(at 203.2 72.3899 0)
+			(effects
+				(font
+					(size 1.27 1.27)
+				)
+				(justify left)
+			)
+		)
+		(property "Value" "100kΩ"
+			(at 203.2 74.9299 0)
+			(effects
+				(font
+					(size 1.27 1.27)
+				)
+				(justify left)
+			)
+		)
+		(property "Footprint" ""
+			(at 198.882 73.66 90)
+			(effects
+				(font
+					(size 1.27 1.27)
+				)
+				(hide yes)
+			)
+		)
+		(property "Datasheet" "~"
+			(at 200.66 73.66 0)
+			(effects
+				(font
+					(size 1.27 1.27)
+				)
+				(hide yes)
+			)
+		)
+		(property "Description" "Resistor"
+			(at 200.66 73.66 0)
+			(effects
+				(font
+					(size 1.27 1.27)
+				)
+				(hide yes)
+			)
+		)
+		(pin "1"
+		)
+		(pin "2"
+		)
+		(instances
+			(project ""
+				(path "/88604d25-498a-4a0c-bf5d-b8ab9ca45bd7/fa45934c-4794-4ba6-bd1a-84173322bb33"
+					(reference "R26")
+					(unit 1)
+				)

Commit message: footprints assigned
Parts:
- C8: footprint (none) -> Capacitor_THT:C_Disc_D5.0mm_W2.5mm_P2.50mm
- IC1: footprint NEOF10N00B -> NEO-F10N-00B:NEOF10N00B
- J2: footprint (none) -> Connector_JST:JST_PH_B2B-PH-K_1x02_P2.00mm_Vertical
- J4, J5: footprint (none) -> Connector_Coaxial:U.FL_Molex_MCRF_73412-0110_Vertical
- Q4: footprint SOT95P240X120-3N -> BSS138:SOT95P240X120-3N
- R16, R17, R26, R28: footprint (none) -> Resistor_THT:R_Axial_DIN0207_L6.3mm_D2.5mm_P7.62mm_Horizontal
Changed lines of the file:
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@@
 			)
 		)
-		(property "Footprint" ""
+		(property "Footprint" "Resistor_THT:R_Axial_DIN0207_L6.3mm_D2.5mm_P7.62mm_Horizontal"
 			(at 215.392 86.36 90)
 			(effects
@@
 			)
 		)
-		(property "Footprint" ""
+		(property "Footprint" "Resistor_THT:R_Axial_DIN0207_L6.3mm_D2.5mm_P7.62mm_Horizontal"
 			(at 35.56 103.378 90)
 			(effects
@@
 			)
 		)
-		(property "Footprint" ""
+		(property "Footprint" "Connector_JST:JST_PH_B2B-PH-K_1x02_P2.00mm_Vertical"
 			(at 269.24 87.63 0)
 			(effects
@@
 			)
 		)
-		(property "Footprint" ""
+		(property "Footprint" "Connector_Coaxial:U.FL_Molex_MCRF_73412-0110_Vertical"
 			(at 134.62 104.14 0)
 			(effects
@@
 			)
 		)
-		(property "Footprint" ""
+		(property "Footprint" "Resistor_THT:R_Axial_DIN0207_L6.3mm_D2.5mm_P7.62mm_Horizontal"
 			(at 95.25 42.672 90)
 			(effects
@@
 			)
 		)
-		(property "Footprint" "SOT95P240X120-3N"
+		(property "Footprint" "BSS138:SOT95P240X120-3N"
 			(at 204.47 191.44 0)
 			(effects
@@
 			)
 		)
-		(property "Footprint" ""
+		(property "Footprint" "Resistor_THT:R_Axial_DIN0207_L6.3mm_D2.5mm_P7.62mm_Horizontal"
 			(at 198.882 73.66 90)
 			(effects
@@
 			)
 		)
-		(property "Footprint" ""
+		(property "Footprint" "Connector_Coaxial:U.FL_Molex_MCRF_73412-0110_Vertical"
 			(at 134.62 87.63 0)
 			(effects
@@
 			)
 		)
-		(property "Footprint" "NEOF10N00B"
+		(property "Footprint" "NEO-F10N-00B:NEOF10N00B"
 			(at 78.74 129.21 0)
 			(effects
@@
 			)
 		)
-		(property "Footprint" ""
+		(property "Footprint" "Capacitor_THT:C_Disc_D5.0mm_W2.5mm_P2.50mm"
 			(at 33.9852 73.66 0)
 			(effects

Commit message: updated to hierarchical labels
Connections:
- net +5V renamed OUT+5V
- net VOUT_3V3: no longer names the net of C8.1, IC1.22 (V_BCKP)
- net VOUT_3V3: no longer Q3.2 (S)
- new net +3V3: Q3.2 (S)
Other:
- sheet GSM_sheet ports: added BAT+, GSM_RXD, GSM_TXD, OUT+5V, VOUT_3V3; removed none

Commit message: last modifications schematic
Connections:
- net +3V3: now also C8.1, IC1.22 (V_BCKP)
Other:
- sheet GSM_sheet ports: added PWRKEY, STATUS; removed none
Changed lines of the file:
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@@
+	(wire
+		(pts
+			(xy 58.42 165.1) (xy 68.58 165.1)
+		)
+		(stroke
+			(width 0)
+			(type default)
+		)
+	)
 	(wire
 		(pts
@@
 	(wire
 		(pts
+			(xy 58.42 167.64) (xy 69.85 167.64)
+		)
+		(stroke
+			(width 0)
+			(type default)
+		)
+	)
+	(wire
+		(pts
 			(xy 31.75 52.07) (xy 39.37 52.07)
 		)
@@
 			(width 0)
 			(type default)
-		)
-	)
-	(global_label "G_DIN"
-		(shape output)
-		(at 213.36 63.5 180)
-		(fields_autoplaced yes)
-		(effects
-			(font
-				(size 1.27 1.27)
-			)
-			(justify right)
-		)
-		(property "Intersheetrefs" "${INTERSHEET_REFS}"
-			(at 204.9319 63.5 0)
-			(hide yes)
-			(show_name no)
-			(do_not_autoplace no)
-			(effects
-				(font
-					(size 1.27 1.27)
-				)
-				(justify right)
-			)
 		)
 	)
@@
 	)
 	(hierarchical_label "TXD"
-		(shape input)
+		(shape output)
 		(at 31.75 52.07 180)
 		(effects
@@
 	(hierarchical_label "G_DIN"
 		(shape input)
-		(at 210.82 59.69 180)
+		(at 213.36 63.5 180)
 		(effects
 			(font
@@
 	)
 	(hierarchical_label "GSM_TXD"
-		(shape input)
+		(shape output)
 		(at 62.23 173.99 0)
+		(effects
+			(font
+				(size 1.27 1.27)
+			)
+			(justify left)
+		)
+	)
+	(hierarchical_label "STATUS"
+		(shape output)
+		(at 68.58 165.1 0)
 		(effects
 			(font
@@
 		)
 	)
+	(hierarchical_label "PWRKEY"
+		(shape input)
+		(at 69.85 167.64 0)
+		(effects
+			(font
+				(size 1.27 1.27)
+			)
+			(justify left)
+		)
+	)
 	(hierarchical_label "+3V3"
 		(shape input)
@@
 	(hierarchical_label "+3V3"
 		(shape input)
-		(at 27.94 57.15 180)
+		(at 29.21 57.15 180)
 		(effects
 			(font
@@
 	)
 	(hierarchical_label "TIMEPULSE"
-		(shape input)
+		(shape output)
 		(at 92.71 57.15 0)
 		(effects
@@
 	)
 	(hierarchical_label "GPS_INT"
-		(shape input)
+		(shape output)
 		(at 86.36 54.61 0)
 		(effects
@@
 			)
 		)
-		(pin "GSM_TXD" input
+		(pin "GSM_TXD" output
 			(at 58.42 173.99 0)
 			(effects
@@
 			(effects
 				(font
+					(size 1.27 1.27)
+				)
+				(justify right)
+			)
+		)
+		(pin "PWRKEY" input
+			(at 58.42 167.64 0)
+			(effects
+				(font
+					(size 1.27 1.27)
+				)
+				(justify right)
+			)
+		)
+		(pin "STATUS" output
+			(at 58.42 165.1 0)
+			(effects
+				(font
