File: PCB/smartBall/STEP_UP.kicad_sch (KiCad schematic)
At the start: 8 parts, among them IC11 TPS61032PWP, IC4 TPS63000IDRCRQ1

Commit message: schematic ready
Parts:
- removed C15, C16: CL31A226MOCLNNC, CAPC3216X100N, symbol CL31A226MOCLNNC:CL31A226MOCLNNC
- added C15: 220µF, symbol Device:C
- added C16: 2.2µF, symbol Device:C
- added L3: 2.2µH, symbol Device:L
- IC11: footprint SOP65P640X120-17N -> TPS61032PWP:SOP65P640X120-17N
- IC4: footprint TPS63000IDRCRQ1 -> TPS63000DRCRQ1:TPS63000IDRCRQ1
Connections:
- net GND: now also C15.2, C16.1
- net OUT+5V: now also C15.1, C16.2
- net at IC4.2 (L2): now also L3.1
- net at IC4.4 (L1): now also L3.2
- net STEP_UP_5_ON renamed LOUDNESS

Commit message: footprints assigned
Parts:
- C14, C15, C16: footprint (none) -> Capacitor_THT:C_Disc_D5.0mm_W2.5mm_P2.50mm
- L2, L3: footprint (none) -> Inductor_THT:L_Axial_L7.0mm_D3.3mm_P10.16mm_Horizontal_Fastron_MICC
- R3, R4: footprint (none) -> Resistor_THT:R_Axial_DIN0207_L6.3mm_D2.5mm_P7.62mm_Horizontal
Changed lines of the file:
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@@
 			)
 		)
-		(property "Footprint" ""
+		(property "Footprint" "Capacitor_THT:C_Disc_D5.0mm_W2.5mm_P2.50mm"
 			(at 257.81 33.9852 0)
 			(effects
@@
 			)
 		)
-		(property "Footprint" ""
+		(property "Footprint" "Resistor_THT:R_Axial_DIN0207_L6.3mm_D2.5mm_P7.62mm_Horizontal"
 			(at 95.25 50.038 90)
 			(effects
@@
 			)
 		)
-		(property "Footprint" ""
+		(property "Footprint" "Inductor_THT:L_Axial_L7.0mm_D3.3mm_P10.16mm_Horizontal_Fastron_MICC"
 			(at 21.59 53.34 0)
 			(effects
@@
 			)
 		)
-		(property "Footprint" ""
+		(property "Footprint" "Capacitor_THT:C_Disc_D5.0mm_W2.5mm_P2.50mm"
 			(at 201.6252 60.96 0)
 			(effects
@@
 			)
 		)
-		(property "Footprint" ""
+		(property "Footprint" "Inductor_THT:L_Axial_L7.0mm_D3.3mm_P10.16mm_Horizontal_Fastron_MICC"
 			(at 214.63 43.18 0)
 			(effects
@@
 			)
 		)
-		(property "Footprint" ""
+		(property "Footprint" "Resistor_THT:R_Axial_DIN0207_L6.3mm_D2.5mm_P7.62mm_Horizontal"
 			(at 38.862 40.64 90)
 			(effects
@@
 			)
 		)
-		(property "Footprint" ""
+		(property "Footprint" "Capacitor_THT:C_Disc_D5.0mm_W2.5mm_P2.50mm"
 			(at 265.43 20.6248 0)
 			(effects

Commit message: new footprints assigned
Parts:
- IC4: footprint TPS63000DRCRQ1:TPS63000IDRCRQ1 -> TPS63000IDRCRQ1:TPS63000IDRCRQ1
Changed lines of the file:
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@@
 			)
 		)
-		(property "Footprint" "TPS63000DRCRQ1:TPS63000IDRCRQ1"
+		(property "Footprint" "TPS63000IDRCRQ1:TPS63000IDRCRQ1"
 			(at 77.47 133.02 0)
 			(hide yes)

Commit message: last modifications schematic
Changed lines of the file:
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@@
 	)
 	(hierarchical_label "+3V3"
-		(shape input)
+		(shape output)
 		(at 35.56 48.26 180)
 		(effects
@@
 	)
 	(hierarchical_label "OUT+5V"
-		(shape input)
+		(shape output)
 		(at 279.4 24.13 90)
 		(effects

Commit message: everything before jlc template
Other:
- moved on the sheet: IC4, L3, R3, R4
