File: PCB/MCU_board/GSM_sheet.kicad_sch (KiCad schematic)
At the start: 28 parts, among them IC2 TXB0104PWR, J6 SIM8055-6-1-14-00-A, J7 FXP612 (u.FL) 1, Q5 BSS138, U2 SIM7000G

Commit message: routing and holes added
Parts:
- TP1: value TestPoint -> USB_DP
- TP2: value TestPoint -> BOOT_CFG
- TP3: value TestPoint -> USB_DM
- TP4: value TestPoint -> USB_VBUS
- TP5: value TestPoint -> MDM_LOG_TX
Connections:
- net BAT+: now also S3.1 (NC)
- no-connect marks 38 -> 37
Changed lines of the file:
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@@
 	)
 	(no_connect
-		(at 251.46 66.04)
-	)
-	(no_connect
 		(at 157.48 123.19)
 	)
@@
 	(wire
 		(pts
+			(xy 251.46 66.04) (xy 251.46 67.31)
+		)
+		(stroke
+			(width 0)
+			(type default)
+		)
+	)
+	(wire
+		(pts
 			(xy 255.27 36.83) (xy 262.89 36.83)
 		)
@@
 			)
 		)
-		(property "Value" "TestPoint"
+		(property "Value" "USB_VBUS"
 			(at 93.98 174.7519 0)
 			(show_name no)
@@
 			)
 		)
-		(property "Value" "TestPoint"
+		(property "Value" "USB_DP"
 			(at 109.22 174.7519 0)
 			(show_name no)
@@
 			)
 		)
-		(property "Value" "TestPoint"
+		(property "Value" "BOOT_CFG"
 			(at 35.56 90.6779 0)
 			(show_name no)
@@
 			)
 		)
-		(property "Value" "TestPoint"
+		(property "Value" "USB_DM"
 			(at 114.3 182.3719 0)
 			(show_name no)
@@
 			)
 		)
-		(property "Value" "TestPoint"
+		(property "Value" "MDM_LOG_TX"
 			(at 88.9 181.1019 0)
 			(show_name no)

Commit message: programming MCU pins
Parts:
- C22: value 100nF -> 1000nF
Changed lines of the file:
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@@
 			)
 		)
-		(property "Value" "100nF"
+		(property "Value" "1000nF"
 			(at 207.01 45.7199 0)
 			(show_name no)

Commit message: everything before jlc template
Parts:
- removed S2, S3: SLW-1276864-4A-D, SLW-1276864-4A-D:SLW12768644AD, symbol SLW-1276864-4A-D:SLW-1276864-4A-D
- added S5: SS14MDP2, SS14MDP2:SS14MDP2, symbol SS14MDP2:SS14MDP2
Connections:
- net BAT+: now also S5.2 (NO_2)
- net OUT+5V: now also S5.1 (NO_1)
- net at D5.2 (K2), FB1.1: now also S5.3 (COM)
- no-connect marks 37 -> 36

Commit message: verifying schematic and 3V8 power for gsm
Parts:
- removed D5: PESD3V3L1BSLZ, PESD3V3L1BSLZ:PESD3V3L1BSLZ, symbol PESD3V3L1BSLZ:PESD3V3L1BSLZ
- removed S5: SS14MDP2, SS14MDP2:SS14MDP2, symbol SS14MDP2:SS14MDP2
- added D1: PESD5V0C1BSFYL, PMEG3005AESFYL, symbol PESD5V0C1BSFYL:PESD5V0C1BSFYL
- C23: value 100µF -> 1000µF
Connections:
- net GND: now also D1.1 (K1)
- net 3V8: now reaches FB1.1
- net 3V8: now also D1.2 (K2)

Commit message: ECR passed
Parts:
- C22: footprint Capacitor_THT:CP_Radial_Tantal_D5.0mm_P2.50mm -> Capacitor_THT:C_Disc_D5.0mm_W2.5mm_P2.50mm
- D1: footprint PMEG3005AESFYL -> PESD5V0C1BSFYL:PMEG3005AESFYL
Changed lines of the file:
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@@
 			)
 		)
-		(property "Description" ""
+		(property "Description" "7 (6 + 1) Position Card Connector NANO SIM Surface Mount, Right Angle Gold"
 			(at 250.19 104.14 0)
 			(hide yes)
@@
 			)
 		)
-		(property "Footprint" "PMEG3005AESFYL"
+		(property "Footprint" "PESD5V0C1BSFYL:PMEG3005AESFYL"
 			(at 245.11 117.78 0)
 			(hide yes)
@@
 			)
 		)
-		(property "Description" ""
+		(property "Description" "Cellular Cat-M, Cat-NB, EDGE, GPRS, LPWA Transceiver Module 850MHz, 900MHz, 1.8GHz, 1.9GHz Antenna Not Included Surface Mount"
 			(at 101.6 107.95 0)
 			(hide yes)
@@
 			)
 		)
-		(property "Footprint" "Capacitor_THT:CP_Radial_Tantal_D5.0mm_P2.50mm"
+		(property "Footprint" "Capacitor_THT:C_Disc_D5.0mm_W2.5mm_P2.50mm"
 			(at 204.1652 48.26 0)
 			(hide yes)

Commit message: routing done
Parts:
- removed C10: CL10B104KO8NNNC, CL10B104KO8NNNC:CAPC1608X90N, symbol CL10B104KO8NNNC:CL10B104KO8NNNC
- added C2: 100nF, symbol Device:C
Connections:
- net GND: now also C2.1
- net SIM_POWER: now also C2.2
Changed lines of the file:
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@@
 	(wire
 		(pts
-			(xy 224.79 86.36) (xy 222.25 86.36)
+			(xy 222.25 86.36) (xy 228.6 86.36)
 		)
 		(stroke
@@
 	(wire
 		(pts
-			(xy 241.3 36.83) (xy 255.27 36.83)
+			(xy 236.22 86.36) (xy 238.76 86.36)
 		)
 		(stroke
@@
 	(wire
 		(pts
-			(xy 219.71 101.6) (xy 238.76 101.6)
+			(xy 241.3 36.83) (xy 255.27 36.83)
 		)
 		(stroke
@@
 	(wire
 		(pts
-			(xy 111.76 35.56) (xy 132.08 35.56)
+			(xy 219.71 101.6) (xy 238.76 101.6)
 		)
 		(stroke
@@
 	(wire
 		(pts
-			(xy 250.19 24.13) (xy 262.89 24.13)
+			(xy 111.76 35.56) (xy 132.08 35.56)
 		)
 		(stroke
@@
 	(wire
 		(pts
-			(xy 233.68 106.68) (xy 242.57 106.68)
+			(xy 250.19 24.13) (xy 262.89 24.13)
 		)
 		(stroke
@@
 	(wire
 		(pts
-			(xy 238.76 86.36) (xy 237.49 86.36)
+			(xy 233.68 106.68) (xy 242.57 106.68)
 		)
 		(stroke
@@
 	)
 	(symbol
+		(lib_id "Device:C")
+		(at 232.41 86.36 270)
+		(unit 1)
+		(body_style 1)
+		(exclude_from_sim no)
+		(in_bom yes)
+		(on_board yes)
+		(in_pos_files yes)
+		(dnp no)
+		(fields_autoplaced yes)
+		(property "Reference" "C2"
+			(at 232.41 78.74 90)
+			(show_name no)
+			(do_not_autoplace no)
+			(effects
+				(font
+					(size 1.27 1.27)
+				)
+			)
+		)
+		(property "Value" "100nF"
+			(at 232.41 81.28 90)
+			(show_name no)
+			(do_not_autoplace no)
+			(effects
+				(font
+					(size 1.27 1.27)
+				)
+			)
+		)
+		(property "Footprint" ""
+			(at 228.6 87.3252 0)
+			(hide yes)
+			(show_name no)
+			(do_not_autoplace no)
+			(effects
+				(font
+					(size 1.27 1.27)
+				)
+			)
+		)
+		(property "Datasheet" ""
+			(at 232.41 86.36 0)
+			(hide yes)
+			(show_name no)
+			(do_not_autoplace no)
+			(effects
+				(font
+					(size 1.27 1.27)
+				)
+			)
+		)
+		(property "Description" "Unpolarized capacitor"
+			(at 232.41 86.36 0)
+			(hide yes)
+			(show_name no)
+			(do_not_autoplace no)
+			(effects
+				(font
+					(size 1.27 1.27)
+				)
+			)
+		)
+		(pin "2"
+		)
+		(pin "1"
+		)
+		(instances
+			(project "MCU_board"
+				(path "/498aac81-136e-41bd-a3ff-29bc0732936d/cfe949ab-0502-475b-aed9-50a88bd6f7c8/ea4c8736-f392-459d-9b84-ce09c609ead2"
+					(reference "C2")
+					(unit 1)
+				)
+			)
+		)
+	)
+	(symbol
 		(lib_id "power:GND")
 		(at 26.67 74.93 0)
@@
 					(unit 1)
 				)
-			)
-		)
-	)
-	(symbol
-		(lib_id "CL10B104KO8NNNC:CL10B104KO8NNNC")
-		(at 224.79 86.36 0)
-		(unit 1)
-		(body_style 1)
-		(exclude_from_sim no)
-		(in_bom yes)
-		(on_board yes)
-		(in_pos_files yes)
-		(dnp no)
-		(fields_autoplaced yes)
-		(property "Reference" "C10"
-			(at 231.14 78.74 0)
-			(show_name no)
-			(do_not_autoplace no)
-			(effects
-				(font
-					(size 1.27 1.27)
-				)
-			)
-		)
-		(property "Value" "CL10B104KO8NNNC"
-			(at 231.14 81.28 0)
-			(show_name no)
-			(do_not_autoplace no)
-			(effects
-				(font
-					(size 1.27 1.27)
-				)
-			)
-		)
-		(property "Footprint" "CL10B104KO8NNNC:CAPC1608X90N"
-			(at 233.68 182.55 0)
-			(hide yes)
-			(show_name no)
-			(do_not_autoplace no)
-			(effects
-				(font
-					(size 1.27 1.27)
-				)
-				(justify left top)
-			)
-		)
-		(property "Datasheet" "https://datasheet.datasheetarchive.com/originals/distributors/Datasheets_SAMA/482ee8b8a1396945e1abac0da9778f7f.pdf"
-			(at 233.68 282.55 0)
-			(hide yes)
-			(show_name no)
-			(do_not_autoplace no)
-			(effects
-				(font
-					(size 1.27 1.27)
-				)
-				(justify left top)
-			)
-		)
-		(property "Description" "Samsung Electro-Mechanics 0603 (1608M) 100nF Multilayer Ceramic Capacitor MLCC 16V dc +/-10% SMD CL10B104KO8NNNC"
-			(at 224.79 86.36 0)
-			(hide yes)
-			(show_name no)
-			(do_not_autoplace no)
-			(effects
-				(font
-					(size 1.27 1.27)
-				)
-			)
-		)
-		(property "Height" "0.9"
-			(at 233.68 482.55 0)
-			(hide yes)
-			(show_name no)
-			(do_not_autoplace no)
-			(effects
-				(font
-					(size 1.27 1.27)
-				)
-				(justify left top)
-			)
-		)
-		(property "Mouser Part Number" "187-CL10B104KO8NNNC"
-			(at 233.68 582.55 0)
-			(hide yes)
-			(show_name no)
-			(do_not_autoplace no)
-			(effects
-				(font
-					(size 1.27 1.27)
-				)
-				(justify left top)
-			)
-		)
-		(property "Mouser Price/Stock" "https://www.mouser.co.uk/ProductDetail/Samsung-Electro-Mechanics/CL10B104KO8NNNC?qs=349EhDEZ59pqoJFRnk4a8w%3D%3D"
-			(at 233.68 682.55 0)
-			(hide yes)
-			(show_name no)
-			(do_not_autoplace no)
-			(effects
-				(font
-					(size 1.27 1.27)
-				)
-				(justify left top)
-			)
-		)
-		(property "Manufacturer_Name" "SAMSUNG"
-			(at 233.68 782.55 0)
-			(hide yes)
-			(show_name no)
-			(do_not_autoplace no)
-			(effects
-				(font
-					(size 1.27 1.27)
-				)
-				(justify left top)
-			)
-		)
-		(property "Manufacturer_Part_Number" "CL10B104KO8NNNC"
-			(at 233.68 882.55 0)
-			(hide yes)
-			(show_name no)
-			(do_not_autoplace no)
-			(effects
-				(font
-					(size 1.27 1.27)
-				)
-				(justify left top)
-			)
-		)
-		(pin "1"
-		)
-		(pin "2"
-		)
-		(instances
-			(project "MCU_board"
-				(path "/498aac81-136e-41bd-a3ff-29bc0732936d/cfe949ab-0502-475b-aed9-50a88bd6f7c8/ea4c8736-f392-459d-9b84-ce09c609ead2"
-					(reference "C10")
-					(unit 1)
-				)

Commit message: DRC passed
Connections:
- net GSM_RXD: no longer IC2.2 (A1), U2.P$10 (RXD)
- net GSM_TXD: no longer IC2.3 (A2), U2.P$9 (TXD)
- net PWRKEY: no longer IC2.4 (A3), U2.P$1 (PWRKEY)
- net STATUS: no longer IC2.5 (A4), U2.P$66 (STATUS)
- new net GSM_RXD_1V8: IC2.2 (A1), U2.P$10 (RXD)
- new net GSM_TXD_1V8: IC2.3 (A2), U2.P$9 (TXD)
- new net PWRKEY_1V8: IC2.4 (A3), U2.P$1 (PWRKEY)
- new net STATUS_1V8: IC2.5 (A4), U2.P$66 (STATUS)
Changed lines of the file:
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@@
 		)
 	)
-	(label "PWRKEY"
+	(label "PWRKEY_1V8"
 		(at 196.85 134.62 180)
 		(effects
@@
 		)
 	)
-	(label "GSM_RXD"
+	(label "GSM_RXD_1V8"
 		(at 191.77 129.54 180)
 		(effects
@@
 		)
 	)
-	(label "PWRKEY"
+	(label "PWRKEY_1V8"
 		(at 30.48 67.31 180)
 		(effects
@@
 		)
 	)
-	(label "GSM_RXD"
+	(label "GSM_RXD_1V8"
 		(at 39.37 113.03 180)
 		(effects
@@
 		)
 	)
-	(label "GSM_TXD"
+	(label "GSM_TXD_1V8"
 		(at 191.77 132.08 180)
 		(effects
@@
 		)
 	)
-	(label "GSM_TXD"
+	(label "GSM_TXD_1V8"
 		(at 39.37 107.95 180)
 		(effects
@@
 		)
 	)
-	(label "STATUS"
+	(label "STATUS_1V8"
 		(at 71.12 46.99 90)
 		(effects
@@
 		)
 	)
-	(label "STATUS"
+	(label "STATUS_1V8"
 		(at 196.85 137.16 180)
 		(effects

Commit message: everything checked
Parts:
- C2: footprint (none) -> Capacitor_THT:C_Disc_D5.0mm_W2.5mm_P2.50mm
Changed lines of the file:
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@@
 			)
 		)
-		(property "Footprint" ""
+		(property "Footprint" "Capacitor_THT:C_Disc_D5.0mm_W2.5mm_P2.50mm"
 			(at 228.6 87.3252 0)
 			(hide yes)
