File: PCB/MCU_board/MCU_board.kicad_sch (KiCad schematic)
At the start: 9 parts, among them IC3 ESP32-S3-WROOM-1-N4R8, J1 DS1013-40SSIB1-B-0

Commit message: routing done
Connections:
- net 3V8: now also J1.2; no longer J1.26
- net ACCEL_INT1: now also J1.20; no longer J1.22
- net ACCEL_INT2: now also J1.22; no longer J1.20
- net MISO: now also J1.6; no longer J1.8
- net MOSI: now also J1.8; no longer J1.6
- net USB_D+: now also J1.37; no longer J1.9
- net USB_D-: now also J1.39; no longer J1.11
- net WCLK: now also J1.26; no longer J1.2
Changed lines of the file:
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@@
+	)
+	(no_connect
+		(at 251.46 50.8)
 	)
 	(no_connect
@@
 	)
 	(no_connect
-		(at 251.46 83.82)
-	)
-	(no_connect
 		(at 105.41 35.56)
 	)
@@
 	)
 	(no_connect
-		(at 251.46 86.36)
+		(at 251.46 48.26)
 	)
 	(no_connect
@@
 		)
 	)
-	(label "MISO"
-		(at 274.32 45.72 0)
-		(effects
-			(font
-				(size 1.27 1.27)
-			)
-			(justify left bottom)
-		)
-	)
-	(label "WCLK"
-		(at 274.32 38.1 0)
-		(effects
-			(font
-				(size 1.27 1.27)
-			)
-			(justify left bottom)
-		)
-	)
 	(label "STATUS"
 		(at 110.49 50.8 0)
@@
 		)
 	)
+	(label "MISO"
+		(at 274.32 43.18 0)
+		(effects
+			(font
+				(size 1.27 1.27)
+			)
+			(justify left bottom)
+		)
+	)
 	(label "STATUS"
 		(at 161.29 166.37 90)
@@
 		)
 	)
+	(label "USB_D+"
+		(at 251.46 83.82 180)
+		(effects
+			(font
+				(size 1.27 1.27)
+			)
+			(justify right bottom)
+		)
+	)
 	(label "G_BCLK"
 		(at 60.96 73.66 180)
@@
 		)
 	)
-	(label "USB_D+"
-		(at 251.46 48.26 180)
-		(effects
-			(font
-				(size 1.27 1.27)
-			)
-			(justify right bottom)
-		)
-	)
 	(label "IMU_INT2"
 		(at 274.32 48.26 0)
@@
 		)
 	)
+	(label "3V8"
+		(at 274.32 38.1 0)
+		(effects
+			(font
+				(size 1.27 1.27)
+			)
+			(justify left bottom)
+		)
+	)
 	(label "G_LRCLK"
 		(at 107.95 68.58 0)
@@
 		)
 	)
+	(label "MOSI"
+		(at 274.32 45.72 0)
+		(effects
+			(font
+				(size 1.27 1.27)
+			)
+			(justify left bottom)
+		)
+	)
 	(label "OUT+5V"
 		(at 251.46 43.18 180)
@@
 		)
 	)
+	(label "WCLK"
+		(at 274.32 68.58 0)
+		(effects
+			(font
+				(size 1.27 1.27)
+			)
+			(justify left bottom)
+		)
+	)
 	(label "I2C_SDA"
 		(at 111.76 63.5 0)
@@
 		)
 	)
+	(label "ACCEL_INT2"
+		(at 274.32 63.5 0)
+		(effects
+			(font
+				(size 1.27 1.27)
+			)
+			(justify left bottom)
+		)
+	)
 	(label "IMU_INT2"
 		(at 110.49 43.18 0)
@@
 		)
 	)
-	(label "3V8"
-		(at 274.32 68.58 0)
-		(effects
-			(font
-				(size 1.27 1.27)
-			)
-			(justify left bottom)
-		)
-	)
 	(label "BAT+"
 		(at 251.46 66.04 180)
@@
 		)
 	)
-	(label "USB_D-"
-		(at 251.46 50.8 180)
-		(effects
-			(font
-				(size 1.27 1.27)
-			)
-			(justify right bottom)
-		)
-	)
 	(label "OUT_N"
 		(at 248.92 68.58 180)
@@
 		)
 	)
+	(label "USB_D-"
+		(at 251.46 86.36 180)
+		(effects
+			(font
+				(size 1.27 1.27)
+			)
+			(justify right bottom)
+		)
+	)
 	(label "G_LRCLK"
 		(at 137.16 167.64 90)
@@
 		)
 	)
-	(label "ACCEL_INT1"
-		(at 274.32 63.5 0)
-		(effects
-			(font
-				(size 1.27 1.27)
-			)
-			(justify left bottom)
-		)
-	)
 	(label "OUT_P"
 		(at 248.92 71.12 180)
@@
 		)
 	)
+	(label "ACCEL_INT1"
+		(at 274.32 60.96 0)
+		(effects
+			(font
+				(size 1.27 1.27)
+			)
+			(justify left bottom)
+		)
+	)
 	(label "GSM_INT"
 		(at 121.92 167.64 90)
@@
 		)
 	)
-	(label "MOSI"
-		(at 274.32 43.18 0)
-		(effects
-			(font
-				(size 1.27 1.27)
-			)
-			(justify left bottom)
-		)
-	)
 	(label "TXD"
 		(at 66.04 43.18 180)
@@
 		)
 	)
-	(label "ACCEL_INT2"
-		(at 274.32 60.96 0)
-		(effects
-			(font
-				(size 1.27 1.27)
-			)
-			(justify left bottom)
-		)
-	)

Commit message: everything checked
Parts:
- added H1, H2, H3, H4: MountingHole, MountingHole:MountingHole_3.2mm_M3_Pad_Via, symbol Mechanical:MountingHole

Commit message: everything done before changing footprints
Connections:
- net GND: now also J1.40
- no-connect marks 18 -> 17
Changed lines of the file:
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@@
-	)
-	(no_connect
-		(at 274.32 86.36)
 	)
 	(no_connect
@@
 	(wire
 		(pts
+			(xy 275.59 86.36) (xy 275.59 87.63)
+		)
+		(stroke
+			(width 0)
+			(type default)
+		)
+	)
+	(wire
+		(pts
 			(xy 45.72 35.56) (xy 45.72 38.1)
 		)
@@
 		(pts
 			(xy 109.22 167.64) (xy 109.22 171.45)
+		)
+		(stroke
+			(width 0)
+			(type default)
+		)
+	)
+	(wire
+		(pts
+			(xy 274.32 86.36) (xy 275.59 86.36)
 		)
 		(stroke
@@
 					(unit 1)
 				)
+			)
+		)
+	)
+	(symbol
+		(lib_id "power:GND")
+		(at 275.59 87.63 0)
+		(unit 1)
+		(body_style 1)
+		(exclude_from_sim no)
+		(in_bom yes)
+		(on_board yes)
+		(in_pos_files yes)
+		(dnp no)
+		(fields_autoplaced yes)
+		(property "Reference" "#PWR05"
+			(at 275.59 93.98 0)
+			(hide yes)
+			(show_name no)
+			(do_not_autoplace no)
+			(effects
+				(font
+					(size 1.27 1.27)
+				)
+			)
+		)
+		(property "Value" "GND"
+			(at 275.59 92.71 0)
+			(show_name no)
+			(do_not_autoplace no)
+			(effects
+				(font
+					(size 1.27 1.27)
+				)
+			)
+		)
+		(property "Footprint" ""
+			(at 275.59 87.63 0)
+			(hide yes)
+			(show_name no)
+			(do_not_autoplace no)
+			(effects
+				(font
+					(size 1.27 1.27)
+				)
+			)
+		)
+		(property "Datasheet" ""
+			(at 275.59 87.63 0)
+			(hide yes)
+			(show_name no)
+			(do_not_autoplace no)
+			(effects
+				(font
+					(size 1.27 1.27)
+				)
+			)
+		)
+		(property "Description" "Power symbol creates a global label with name \"GND\" , ground"
+			(at 275.59 87.63 0)
+			(hide yes)
+			(show_name no)
+			(do_not_autoplace no)
+			(effects
+				(font
+					(size 1.27 1.27)
+				)
+			)
+		)
+		(pin "1"
+		)
+		(instances
+			(project "MCU_board"
+				(path "/498aac81-136e-41bd-a3ff-29bc0732936d"
+					(reference "#PWR05")
+					(unit 1)
+				)
