File: PCB/MCU_board/Stationary.kicad_sch (KiCad schematic)
At the start: 11 parts, among them IC1 NEO-F10N-00B, IC6 4259-63, IC8 MAX98357AETE+T, J4 FXP612 (u.FL) 2, J5 FXP612 (u.FL) 1, Q3 Si2323DDS-T1-GE3

Commit message: modified gnd
Parts:
- removed IC8: MAX98357AETE+T, MAX98357AETE+T:QFN50P300X300X80-17N, symbol MAX98357AETE+T:MAX98357AETE+T
- removed R16, R26: 100kΩ, Resistor_THT:R_Axial_DIN0207_L6.3mm_D2.5mm_P7.62mm_Horizontal, symbol Device:R
- added IC4: MAX98357AETE+T, MAX98357AETE+T:QFN50P300X300X80-17N, symbol MAX98357AETE+T:MAX98357AETE+T
- added J2: Conn_02x04_Counter_Clockwise, Connector_PinHeader_2.54mm:PinHeader_2x04_P2.54mm_Vertical, symbol Connector_Generic:Conn_02x04_Counter_Clockwise
- added R1: 10kΩ, Resistor_SMD:R_0603_1608Metric, symbol Device:R
- added R2: 100kΩ, Resistor_SMD:R_0603_1608Metric, symbol Device:R
- C8: footprint Capacitor_THT:C_Disc_D5.0mm_W2.5mm_P2.50mm -> Capacitor_SMD:CP_Elec_6.3x5.4
- Q3: footprint Si2323DDS-T1-GE3:SOT95P237X112-3N -> Package_TO_SOT_SMD:SOT-23
- R17, R28: footprint Resistor_THT:R_Axial_DIN0207_L6.3mm_D2.5mm_P7.62mm_Horizontal -> Resistor_SMD:R_0603_1608Metric
Connections:
- net +3V3: now also J2.1 (Pin_1)
- net GND: now also IC4.11 (GND_2), IC4.15 (GND_3), IC4.17 (THERMAL_PAD), IC4.3 (GND_1), J2.5 (Pin_5), R1.2
- net G_BCLK: now also IC4.16 (BCLK)
- net G_DIN: now also IC4.1 (DIN)
- net G_LRCLK: now also IC4.14 (LRCLK)
- net LOUDNESS: now also R2.2
- net OUT+5V: now also IC4.7 (VDD_1), IC4.8 (VDD_2)
- net OUTP: now also IC4.9 (OUTP)
- net OUT_N: now also IC4.10 (OUTN)
- net RXD: now also J2.3 (Pin_3)
- net TIMEPULSE: now also J2.4 (Pin_4)
- net TXD: now also J2.2 (Pin_2)
- new net: IC4.2 (GAIN_SLOT), R1.1
- new net: IC4.4 (~{SD_MODE}), R2.1
- no-connect marks 15 -> 18
Other:
- sheet GSM_sheet ports: added none; removed 3V8
